File: heater.kicad_sch (KiCad schematic)
At the start: 0 parts

Commit message: Schematic Completed
Parts:
- added J10, J15: C8465, symbol Connector:Screw_Terminal_01x02
- added J16, J17: Screw_Terminal_01x02, symbol Connector:Screw_Terminal_01x02
- added Q3: AO3406, symbol Simulation_SPICE:NMOS
- added R35: 1k, symbol Device:R_Small
- added R36: 330, symbol Device:R_Small
- added TP1, TP2: relay_trigger_TP, Connector_PinHeader_2.54mm:PinHeader_1x01_P2.54mm_Horizontal, symbol Connector:TestPoint
- added U10, U11, U9: G5NB-1A-E DC12, Package_SIP:SIP4_Sharp-SSR_P7.62mm_Straight, symbol Relay_SolidState:S102S01
Connections:
- new net: J10.1 (Pin_1), J10.2 (Pin_2), J17.1 (Pin_1), J17.2 (Pin_2), U10.1, U11.1, U9.1
- new net: Q3.1 (D), TP1.1, U10.4, U11.4, U9.4
- new net: Q3.3 (S), R35.1
- new net: J15.1 (Pin_1), J15.2 (Pin_2), J16.1 (Pin_1), J16.2 (Pin_2), U10.2, U11.2, U9.2
- new net +12V: TP2.1, U10.3, U11.3, U9.3
- new net GND: R35.2, R36.2
- new net heater: Q3.2 (G), R36.1
Other:
- note added: "Screw terminal"
- note added: "ssr relay"
