File: outputs.kicad_sch (KiCad schematic)
At the start: 0 parts

Commit message: Power Section done + added backup lipo
Parts:
- added BZ1: Buzzer, symbol Device:Buzzer
- added D10: FAULT_LED, symbol Device:LED
- added D11: BUSY_LED, symbol Device:LED
- added D12: CONNECTIVITY_LED, symbol Device:LED
- added D4, D5, D6, D7, D8: 1N4001, Diode_THT:D_DO-41_SOD81_P10.16mm_Horizontal, symbol Diode:1N4001
- added D9: LED_PWR, symbol Device:LED
- added J12: Water_Pump, symbol Connector_Generic:Conn_01x02
- added J13: Fan_Continous, symbol Connector_Generic:Conn_01x02
- added J2: mist, symbol Connector_Generic:Conn_01x02
- added J3: Led, symbol Connector_Generic:Conn_01x02
- added J8: Fan_Exhaust, symbol Connector_Generic:Conn_01x02
- added Q1, Q2, Q3, Q4, Q5, Q6: AO3406, symbol Simulation_SPICE:NMOS
- added R10, R11, R12, R13, R14, R15: 1K, symbol Device:R
- added R2, R5, R6, R7, R8, R9: 10K, symbol Device:R
Connections:
- new net: D12.1 (K), R15.1
- new net: D5.2 (A), J12.2 (Pin_2), Q2.1 (D)
- new net: D10.1 (K), R13.1
- new net: D8.2 (A), J8.2 (Pin_2), Q6.1 (D)
- new net: BZ1.2 (+), D4.2 (A), R10.1
- new net: Q1.1 (D), R10.2
- new net: D7.2 (A), J13.2 (Pin_2), Q5.1 (D)
- new net: D6.2 (A), Q4.1 (D), R11.1
- new net: J2.2 (Pin_2), R11.2
- new net: D11.1 (K), R14.1
- new net: J3.2 (Pin_2), Q3.1 (D)
- new net: D9.1 (K), R12.1
- new net +12V: BZ1.1 (-), D4.1 (K), D5.1 (K), D6.1 (K), D7.1 (K), D8.1 (K), D9.2 (A), J12.1 (Pin_1), J13.1 (Pin_1), J2.1 (Pin_1), J3.1 (Pin_1), J8.1 (Pin_1)
- new net BUSY_LED: D11.2 (A)
- new net BUZ_PIN: Q1.2 (G), R5.2
- new net CON_LED: D12.2 (A)
- new net FAN_CON_PIN: Q5.2 (G), R8.2
- new net FAN_EXHAUST_PIN: Q6.2 (G), R9.2
- new net FAULT_LED: D10.2 (A)
- new net GND: Q1.3 (S), Q2.3 (S), Q3.3 (S), Q4.3 (S), Q5.3 (S), Q6.3 (S), R12.2, R13.2, R14.2, R15.2, R2.1, R5.1, R6.1, R7.1, R8.1, R9.1
- new net LED_PIN: Q3.2 (G), R6.2
- new net MIST_PIN: Q4.2 (G), R7.2
- new net WATER_PUMP_PIN: Q2.2 (G), R2.2
Other:
- note added: "Outputs"

Commit message: Schematic Completed
Parts:
- removed R15: 1K, symbol Device:R
- added D3: LED, symbol Device:LED
- added D6: 1N4001, Diode_THT:D_DO-41_SOD81_P10.16mm_Horizontal, symbol Diode:1N4001
- added J10 (x3), J15: C8465, symbol Connector:Screw_Terminal_01x02
- added J10: Display, symbol Connector_Generic:Conn_01x04
- added J11: Rotary_Encoder, symbol Connector_Generic:Conn_01x05
- added J16, J17: Screw_Terminal_01x02, symbol Connector:Screw_Terminal_01x02
- added J4: Water_Level, symbol Connector_Generic:Conn_01x03
- added J7: Temp, symbol Connector_Generic:Conn_01x03
- added J9: Temp2, symbol Connector_Generic:Conn_01x03
- added Q3 (x3): AO3406, symbol Simulation_SPICE:NMOS
- added R15 (x2): 1K, symbol Device:R
- added R35 (x3): 1k, symbol Device:R_Small
- added R36 (x3): 330, symbol Device:R_Small
- added TP1, TP2: relay_trigger_TP, Connector_PinHeader_2.54mm:PinHeader_1x01_P2.54mm_Horizontal, symbol Connector:TestPoint
- added U10, U11, U9 (x2): G5NB-1A-E DC12, Package_SIP:SIP4_Sharp-SSR_P7.62mm_Straight, symbol Relay_SolidState:S102S01
Connections:
- net +12V: now also D6.1 (K), J10.1 (Pin_1), TP2.1, U10.3, U11.3, U9.3, U9.3
- net GND: now also J10.1 (Pin_1), J11.1 (Pin_1), J4.1 (Pin_1), J7.1 (Pin_1), J9.1 (Pin_1), R15.2, R15.2, R35.2, R35.2, R35.2, R36.2, R36.2, R36.2
- net at D12.1 (K): now also R15.1
- new net: J10.1 (Pin_1), J10.2 (Pin_2), J17.1 (Pin_1), J17.2 (Pin_2), U10.1, U11.1, U9.1
- new net: Q3.3 (S), R35.1 (x3)
- new net: J15.1 (Pin_1), J15.2 (Pin_2), J16.1 (Pin_1), J16.2 (Pin_2), U10.2, U11.2, U9.2
- new net: Q3.1 (D), TP1.1, U10.4, U11.4, U9.4
- new net: D3.1 (K), R15.1
- new net: J10.1 (Pin_1), U9.1
- new net: J10.2 (Pin_2), U9.2
- new net: D6.2 (A), J10.2 (Pin_2), Q3.1 (D)
- new net: Q3.1 (D), U9.4
- new net +3.3V: J10.2 (Pin_2), J11.2 (Pin_2), J4.2 (Pin_2), J7.2 (Pin_2), J9.2 (Pin_2)
- new net IO_LED: D3.2 (A)
- new net ROTARY_CLK: J11.4 (Pin_4)
- new net ROTARY_DATA: J11.5 (Pin_5)
- new net ROT_SW: J11.3 (Pin_3)
- new net SCL: J10.4 (Pin_4)
- new net SDA: J10.3 (Pin_3)
- new net TEMP1_DATA: J7.3 (Pin_3)
- new net TEMP2_DATA: J9.3 (Pin_3)
- new net WATER_LEVEL_DATA: J4.3 (Pin_3)
- new net heater: Q3.2 (G), R36.1
- new net turner: Q3.2 (G), Q3.2 (G), R36.1, R36.1
Other:
- note added: "HEATER"
- note added: "JST connectors"
- note added: "LEDS"
- note added: "Optional DC motor"
- note added: "Primary AC"
- note added: "Screw terminal"
- note added: "Sensors/Inputs"
- note added: "TURNER"
- note added: "ssr relay"
- moved on the sheet: BZ1, D4, D5, D6, D7, D8, J12, J13, J2, J3, J8, Q1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
