File: turner.kicad_sch (KiCad schematic)
At the start: 0 parts

Commit message: Schematic Completed
Parts:
- added D6: 1N4001, Diode_THT:D_DO-41_SOD81_P10.16mm_Horizontal, symbol Diode:1N4001
- added J10 (x2): C8465, symbol Connector:Screw_Terminal_01x02
- added Q3 (x2): AO3406, symbol Simulation_SPICE:NMOS
- added R35 (x2): 1k, symbol Device:R_Small
- added R36 (x2): 330, symbol Device:R_Small
- added U9: G5NB-1A-E DC12, Package_SIP:SIP4_Sharp-SSR_P7.62mm_Straight, symbol Relay_SolidState:S102S01
Connections:
- new net: Q3.3 (S), R35.1 (x2)
- new net: D6.2 (A), J10.2 (Pin_2), Q3.1 (D)
- new net: Q3.1 (D), U9.4
- new net: J10.1 (Pin_1), U9.1
- new net: J10.2 (Pin_2), U9.2
- new net +12V: D6.1 (K), J10.1 (Pin_1), U9.3
- new net GND: R35.2, R35.2, R36.2, R36.2
- new net turner: Q3.2 (G), Q3.2 (G), R36.1, R36.1
Other:
- note added: "Optional DC motor"
- note added: "Primary AC"
