File: Capibator_PCB.kicad_pcb (KiCad board)
At the start: 2 copper layers, 118 parts, among them J1 FTDI, J10 mist, J11 Led, J12 Water_Level, J13 Main_Input_Jack, J14 Battery, J15 Display, J16 Rotary_Encoder, J17 Temp, J18 Temp2, J19 Water_Pump, J2 LED, J20 Conn_01x04_Socket, J21 extra, J3 C8465, J4 C8465, J5 Screw_Terminal_01x02, J6 C8465, J7 Screw_Terminal_01x02, J8 Fan_Exhaust, J9 Fan_Continous, Q10 AO3406, Q2 AO3406, Q3 AO3406, Q4 AO3406, Q5 AO3406, Q6 AO3406, Q7 SI2301, Q8 AO3406, Q9 AO3406, SW1 SW_MEC_5G, SW2 SW_MEC_5G, SW4 SW, U10 G5NB-1A-E DC12, U2 ESP32-WROOM-32, U5 PCF8574, U6 LM7805_TO220, U7 TP4056, U8 DS1307+, U9 G5NB-1A-E DC12, Y1 32.768kHz Quartz Crystal

Commit message: started pcb
Parts:
- removed J11: Led, LED_SMD:LED_0805_2012Metric
- removed U10: G5NB-1A-E DC12, Package_SIP:SIP4_Sharp-SSR_P7.62mm_Straight
- added D1: 1N5819WS, Diode_SMD:D_SOD-323, F.Cu at (144.6, 76.8)
- added K1: G5NB-1A-E DC12, G5NB-1A-E_DC12:RELAY_G5NB-1A_DC5_OMR, F.Cu at (120.4, 60.3)
- added U3: AMS1117-5.0, Package_TO_SOT_SMD:SOT-223-3_TabPin2, F.Cu at (133.4, 62.7)
- D12: footprint Diode_SMD:D_0805_2012Metric -> Diode_THT:D_DO-41_SOD81_P10.16mm_Horizontal
- U1: value ~ -> TPS63070RNMR; footprint Package_DFN_QFN:TDFN-8-1EP_2x2mm_P0.5mm_EP0.8x1.2mm -> TPS63070RNMR:VREG_TPS63070RNMR
- U6: value LM7805_TO220 -> MAX17048G_T10; footprint Package_TO_SOT_THT:TO-220F-3_Horizontal_TabDown -> MAX17048G_T10:SON50P200X200X80-9N
- U9: footprint Package_SIP:SIP4_Sharp-SSR_P7.62mm_Straight -> G5NB-1A-E_DC12:RELAY_G5NB-1A_DC5_OMR
- moved R1 114.2 mm to (112.4, 99.2)
- moved R8 92.9 mm to (130.0, 79.1)
- moved D3 87.8 mm to (184.8, 114.5), turned to 90 degrees
- moved D6 87.7 mm to (184.9, 122.5), turned to 90 degrees
- moved U9 86.7 mm to (107.5, 60.1), turned to 180 degrees
- moved L1 86.5 mm to (155.1, 62.3)
- moved R37 86.3 mm to (150.4, 71.3), turned to 180 degrees
- moved R11 84.3 mm to (153.3, 115.4), turned to 180 degrees
- moved C17 84.2 mm to (161.6, 65.9)
- moved C18 84.2 mm to (162.9, 65.9)
- moved C19 84.2 mm to (164.1, 65.9)
- moved C21 84.2 mm to (165.4, 65.9)
- moved R30 84.2 mm to (160.3, 65.6)
- moved R25 84.2 mm to (160.3, 67.5)
- moved R12 84.1 mm to (153.3, 116.9), turned to 180 degrees
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Connections:
- L1 pad 1: Net-(U4-L1) -> Net-(U1-L2)
- L1 pad 2: Net-(U4-L2) -> Net-(U1-L1)
- R17 pad 1: Net-(U1-QSTART) -> Net-(U6-QSTRT)
- R18 pad 1: +3.3V -> /MCU/SDA
- R18 pad 2: /MCU/SDA -> +3.3V
- R22 pad 2: Net-(U1-ALERT) -> Net-(U6-~{ALERT})
- U1 pad 1: GND -> unconnected-(U1-PS/SYNC-Pad1)
- U1 pad 2: MCU_BAT -> unconnected-(U1-PG-Pad2)
- U1 pad 3: Net-(JP1-C) -> unconnected-(U1-VAUX-Pad3)
- U1 pad 4: (no net) -> unconnected-(U1-GND-Pad4)
- U1 pad 5: Net-(U1-ALERT) -> unconnected-(U1-FB-Pad5)
- U1 pad 6: Net-(U1-QSTART) -> unconnected-(U1-FB2-Pad6)
- U1 pad 9: (no net) -> Net-(U1-L2)
- U4 pad 9: Net-(U4-L2) -> unconnected-(U4-L2-Pad9)
- U6 pad 1: +12V -> GND
- U6 pad 2: GND -> MCU_BAT
- U6 pad 3: +5V -> Net-(JP1-C)
- U9 pad 1: Net-(J3-Pin_2) -> Net-(Q3-D)
- U9 pad 3: +12V -> Net-(J3-Pin_2)
- U9 pad 4: Net-(Q3-D) -> +12V
Other:
- board text added: "buttons shouldn't be ground."

Commit message: first revision of pcb ready. very crude.. needs another looky
Parts:
- removed JP1: Jumper_3_Bridged12, Jumper:SolderJumper-3_P1.3mm_Bridged2Bar12_Pad1.0x1.5mm_NumberLabels
- removed JP3: Jumper_2_Open, Jumper:SolderJumper-2_P1.3mm_Open_Pad1.0x1.5mm
- removed SW4: SW, Button_Switch_SMD:Nidec_Copal_CAS-120A
- removed U4: ~, Package_DFN_QFN:TDFN-8-1EP_2x2mm_P0.5mm_EP0.8x1.2mm
- added C10: 10u, Capacitor_SMD:C_0805_2012Metric, F.Cu at (122.4, 101.0)
- C1, C12, C13, C14, C15, C2, C20, C3, C4, C5, C6, C7, C8, C9: footprint Capacitor_SMD:C_0402_1005Metric -> Capacitor_SMD:C_0805_2012Metric
- C17, C18, C19, C21: footprint Capacitor_SMD:C_0402_1005Metric -> Resistor_SMD:R_0805_2012Metric
- D1: footprint Diode_SMD:D_SOD-323 -> Diode_SMD:D_0805_2012Metric
- D12: footprint Diode_THT:D_DO-41_SOD81_P10.16mm_Horizontal -> Diode_SMD:D_0603_1608Metric
- J1: footprint Connector_PinHeader_2.54mm:PinHeader_1x06_P2.54mm_Horizontal -> Connector_PinHeader_2.54mm:PinHeader_1x06_P2.54mm_Vertical
- J16: value Rotary_Encoder -> Conn_01x05; footprint Connector_JST:JST_GH_SM03B-GHS-TB_1x03-1MP_P1.25mm_Horizontal -> Connector_JST:JST_GH_SM05B-GHS-TB_1x05-1MP_P1.25mm_Horizontal
- R1, R10, R11, R12, R13, R14, R15, R16, R17, R18, R19, R20, R21, R22, R23, R24, R25, R26, R27, R28, R29, R30, R31, R32, R35, R38, R39, R41, R5, R6, R8, R9: footprint Resistor_SMD:R_0201_0603Metric -> Resistor_SMD:R_0805_2012Metric
- R3, R4: footprint Resistor_SMD:R_0201_0603Metric -> Capacitor_SMD:C_0805_2012Metric
- SW1, SW2: value SW_MEC_5G -> SW_Omron_B3FS; footprint Button_Switch_SMD:SW_SPST_B3U-1000P -> Button_Switch_SMD:SW_SPST_Omron_B3FS-100xP
- U8: footprint Package_DIP:DIP-8_W7.62mm -> DS1307ZTR:21-0041B_8
- moved C3 43.9 mm to (116.7, 100.7), turned to 180 degrees
- moved C17 37.6 mm to (129.3, 85.1), turned to 90 degrees
- moved C18 36.8 mm to (131.5, 85.1), turned to 90 degrees
- moved C19 36.0 mm to (133.7, 85.1), turned to 90 degrees
- moved C21 35.2 mm to (135.9, 85.1), turned to 90 degrees
- moved Y1 35.1 mm to (145.4, 72.1)
- moved R23 32.4 mm to (132.7, 70.8), turned to -90 degrees
- moved C4 31.5 mm to (148.5, 75.9), turned to 90 degrees
- moved C9 31.4 mm to (150.7, 75.9), turned to 90 degrees
- moved R25 31.0 mm to (132.7, 81.5)
- moved R30 30.0 mm to (134.9, 81.5), turned to 90 degrees
- moved R22 25.5 mm to (137.8, 70.8), turned to -90 degrees
- moved L1 25.3 mm to (141.1, 83.4)
- moved C12 24.1 mm to (162.1, 74.3)
- moved C14 24.0 mm to (132.7, 77.9), turned to -90 degrees
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Connections:
- C1 pad 1: Net-(JP2-B) -> /MCU/TPS_VIN
- C13 pad 1: Net-(JP2-B) -> /MCU/TPS_VIN
- C14 pad 1: Net-(U4-VAUX) -> /MCU/TPS_VAUX
- C2 pad 1: Net-(JP2-B) -> /MCU/TPS_VIN
- C8 pad 1: Net-(JP2-B) -> /MCU/TPS_VIN
- J14 pad 2: Net-(SW4-B) -> MCU_BAT
- J20 pad 3: /MCU/P_IO_4 -> /MCU/P_IO_7
- JP2 pad 2: Net-(JP2-B) -> /MCU/TPS_VIN
- R23 pad 1: Net-(JP2-B) -> /MCU/TPS_VIN
- R24 pad 1: Net-(JP2-B) -> /MCU/TPS_VIN
- R25 pad 1: Net-(U4-FB) -> /MCU/TPS_FB
- R30 pad 2: Net-(U4-FB) -> /MCU/TPS_FB
- SW1 pad 2: GND -> /MCU/GPIO0
- SW2 pad 2: GND -> /MCU/RESET
- U1 pad 1: unconnected-(U1-PS/SYNC-Pad1) -> /MCU/PS
- U1 pad 10: unconnected-(U1-PGND-Pad10) -> GND
- U1 pad 12_13: unconnected-(U1-VIN-Pad12_13) -> /MCU/TPS_VIN
- U1 pad 14: unconnected-(U1-EN-Pad14) -> /MCU/EN
- U1 pad 15: unconnected-(U1-VSEL-Pad15) -> GND
- U1 pad 2: unconnected-(U1-PG-Pad2) -> GND
- U1 pad 3: unconnected-(U1-VAUX-Pad3) -> /MCU/TPS_VAUX
- U1 pad 4: unconnected-(U1-GND-Pad4) -> GND
- U1 pad 5: unconnected-(U1-FB-Pad5) -> /MCU/TPS_FB
- U1 pad 6: unconnected-(U1-FB2-Pad6) -> GND
- U1 pad 7_8: unconnected-(U1-VOUT-Pad7_8) -> +3.3V
- U5 pad 10: /MCU/P_IO_4 -> /MCU/P_IO_7
- U6 pad 3: Net-(JP1-C) -> MCU_BAT
Routing:
- net GND: track 0.00 -> 469.8 mm, vias 0 -> 34
- net +3.3V: track 0.00 -> 311.2 mm, vias 0 -> 23
- net +12V: track 0.00 -> 242.7 mm, vias 0 -> 8
- net /MCU/SDA: track 0.00 -> 142.4 mm, vias 0 -> 7
- net /MCU/SCL: track 0.00 -> 141.9 mm, vias 0 -> 6
- net /MCU/LED_PIN: track 0.00 -> 126.8 mm, vias 0 -> 6
- net /MCU/turner: track 0.00 -> 105.3 mm
- net /MCU/GPIO2: track 0.00 -> 88.8 mm, vias 0 -> 8
- net /MCU/FAN_CON_PIN: track 0.00 -> 87.2 mm, vias 0 -> 4
- net /MCU/BUZ_PIN: track 0.00 -> 84.2 mm, vias 0 -> 8
- net /MCU/WATER_LEVEL_DATA: track 0.00 -> 83.2 mm, vias 0 -> 2
- net /MCU/RESET: track 0.00 -> 82.2 mm, vias 0 -> 8
- net /MCU/ROT_SW: track 0.00 -> 73.5 mm, vias 0 -> 2
- net /MCU/ROTARY_DATA: track 0.00 -> 67.6 mm, vias 0 -> 2
- net /MCU/ROTARY_CLK: track 0.00 -> 67.2 mm, vias 0 -> 2
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Other:
- board text removed: "buttons shouldn't be ground."
