File: MCU.kicad_sch (KiCad schematic)
At the start: 117 parts, among them J10 mist, J11 Led, J12 Water_Level, J13 Main_Input_Jack, J14 Battery, J15 Display, J16 Rotary_Encoder, J17 Temp, J18 Temp2, J19 Water_Pump, J2 FTDI, J20 Conn_01x04_Socket, J21 extra, J3 C8465, J4 C8465, J5 Screw_Terminal_01x02, J6 C8465, J7 Screw_Terminal_01x02, J8 Fan_Exhaust, J9 Fan_Continous, Q10 AO3406, Q2 AO3406, Q3 AO3406, Q4 AO3406, Q5 AO3406, Q6 AO3406, Q7 SI2301, Q8 AO3406, Q9 AO3406, SW1 SW_MEC_5G, SW2 SW_MEC_5G, SW4 SW, U1 ESP32-WROOM-32, U10 G5NB-1A-E DC12, U4 TP4056, U5 PCF8574, U6 LM7805_TO220, U8 DS1307+, U9 G5NB-1A-E DC12, Y1 32.768kHz Quartz Crystal

Commit message: started pcb and basic alignment
Parts:
- removed J11: Led, LED_SMD:LED_0805_2012Metric, symbol Connector_Generic:Conn_01x02
- added J2: LED, Connector_JST:JST_GH_SM02B-GHS-TB_1x02-1MP_P1.25mm_Horizontal, symbol Connector_Generic:Conn_01x02
Connections:
- net +12V: now also J2.1 (Pin_1)
- net at Q8.1 (D): now also J2.2 (Pin_2)
Changed lines of the file:
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@@
   (junction (at 480.06 73.025) (diameter 0) (color 0 0 0 0)
   )
+  (junction (at 179.07 198.12) (diameter 0) (color 0 0 0 0)
+  )
   (junction (at 219.71 194.31) (diameter 0) (color 0 0 0 0)
   )
@@
     (stroke (width 0) (type default))
   )
+  (wire (pts (xy 179.07 196.85) (xy 179.07 198.12))
+    (stroke (width 0) (type default))
+  )
   (wire (pts (xy 237.49 189.23) (xy 246.38 189.23))
     (stroke (width 0) (type default))
@@
     (stroke (width 0) (type default))
   )
+  (wire (pts (xy 178.435 198.12) (xy 179.07 198.12))
+    (stroke (width 0) (type default))
+  )
   (wire (pts (xy 445.77 46.355) (xy 464.82 46.355))
     (stroke (width 0) (type default))
@@
     (stroke (width 0) (type default))
   )
+  (wire (pts (xy 173.355 198.12) (xy 172.72 198.12))
+    (stroke (width 0) (type default))
+  )
   (wire (pts (xy 172.72 203.2) (xy 172.72 198.12))
     (stroke (width 0) (type default))
@@
     (stroke (width 0) (type default))
   )
+  (wire (pts (xy 179.07 198.12) (xy 182.88 198.12))
+    (stroke (width 0) (type default))
+  )
   (wire (pts (xy 501.65 65.405) (xy 508 65.405))
     (stroke (width 0) (type default))
@@
     (stroke (width 0) (type default))
   )
-  (wire (pts (xy 173.99 198.12) (xy 172.72 198.12))
-    (stroke (width 0) (type default))
-  )
   (wire (pts (xy 231.775 63.5) (xy 236.855 63.5))
     (stroke (width 0) (type default))
@@
     (stroke (width 0) (type default))
   )
-  (wire (pts (xy 179.07 198.12) (xy 182.88 198.12))
-    (stroke (width 0) (type default))
-  )
   (wire (pts (xy 525.78 56.515) (xy 525.78 60.325))
     (stroke (width 0) (type default))
@@
     (effects (font (size 1.27 1.27)) (justify left bottom))
   )
-  (label "EN" (at 179.07 198.12 0) (fields_autoplaced)
+  (label "EN" (at 179.07 196.85 0) (fields_autoplaced)
     (effects (font (size 1.27 1.27)) (justify left bottom))
   )
@@
     )
   )
-  (symbol (lib_id "Connector_Generic:Conn_01x02") (at 471.17 53.975 0) (unit 1)
-    (in_bom yes) (on_board yes) (dnp no) (fields_autoplaced)
-    (property "Reference" "J11" (at 473.71 53.975 0)
-      (effects (font (size 1.27 1.27)) (justify left))
-    )
-    (property "Value" "Led" (at 473.71 56.515 0)
-      (effects (font (size 1.27 1.27)) (justify left))
-    )
-    (property "Footprint" "LED_SMD:LED_0805_2012Metric" (at 471.17 53.975 0)
-      (effects (font (size 1.27 1.27)) hide)
-    )
-    (property "Datasheet" "~" (at 471.17 53.975 0)
-      (effects (font (size 1.27 1.27)) hide)
-    )
-    (pin "1")
-    (pin "2")
-    (instances
-      (project "Capibator_PCB"
-        (path "/314af396-fc31-4fe3-9f85-bbd0c4bf0b50/6d26da2f-4df7-46b4-abe0-c85ffa1a5908"
-          (reference "J11") (unit 1)
-        )
-      )
-    )
-  )
   (symbol (lib_id "Device:L") (at 193.04 180.34 90) (unit 1)
     (in_bom yes) (on_board yes) (dnp no) (fields_autoplaced)
@@
     )
   )
-  (symbol (lib_id "Device:R_Small") (at 176.53 198.12 90) (unit 1)
+  (symbol (lib_id "Device:R_Small") (at 175.895 198.12 90) (unit 1)
     (in_bom yes) (on_board yes) (dnp no)
-    (property "Reference" "R23" (at 176.53 193.04 90)
+    (property "Reference" "R23" (at 175.895 193.04 90)
       (effects (font (size 1.27 1.27)) hide)
     )
-    (property "Value" "10k" (at 176.53 198.12 90)
+    (property "Value" "10k" (at 175.895 196.215 90)
       (effects (font (size 1 1)))
     )
-    (property "Footprint" "Resistor_SMD:R_0201_0603Metric" (at 176.53 198.12 0)
+    (property "Footprint" "Resistor_SMD:R_0201_0603Metric" (at 175.895 198.12 0)
       (effects (font (size 1.27 1.27)) hide)
     )
-    (property "Datasheet" "~" (at 176.53 198.12 0)
+    (property "Datasheet" "~" (at 175.895 198.12 0)
       (effects (font (size 1.27 1.27)) hide)
     )
@@
         )
       )
+    )
+  )
+  (symbol (lib_id "Connector_Generic:Conn_01x02") (at 471.17 53.975 0) (unit 1)
+    (in_bom yes) (on_board yes) (dnp no) (fields_autoplaced)
+    (property "Reference" "J2" (at 473.71 53.975 0)
+      (effects (font (size 1.27 1.27)) (justify left))
+    )
+    (property "Value" "LED" (at 473.71 56.515 0)
+      (effects (font (size 1.27 1.27)) (justify left))
+    )
+    (property "Footprint" "Connector_JST:JST_GH_SM02B-GHS-TB_1x02-1MP_P1.25mm_Horizontal" (at 471.17 53.975 0)
+      (effects (font (size 1.27 1.27)) hide)
+    )
+    (property "Datasheet" "~" (at 471.17 53.975 0)
+      (effects (font (size 1.27 1.27)) hide)
+    )
+    (pin "1")
+    (pin "2")
+    (instances
+      (project "Capibator_PCB"
+        (path "/314af396-fc31-4fe3-9f85-bbd0c4bf0b50/6d26da2f-4df7-46b4-abe0-c85ffa1a5908"
+          (reference "J2") (unit 1)
+        )
+      )

Commit message: started pcb
Parts:
- removed D12: 1N5819, Diode_SMD:D_0805_2012Metric, symbol Diode:1N5819
- removed J5, J7: Screw_Terminal_01x02, TerminalBlock:TerminalBlock_Altech_AK300-2_P5.00mm, symbol Connector:Screw_Terminal_01x02
- removed JP3: Jumper_2_Open, Jumper:SolderJumper-2_P1.3mm_Open_Pad1.0x1.5mm, symbol Jumper:Jumper_2_Open
- removed U1: ~, Package_DFN_QFN:TDFN-8-1EP_2x2mm_P0.5mm_EP0.8x1.2mm, symbol Custom:MAX17048
- removed U10: G5NB-1A-E DC12, Package_SIP:SIP4_Sharp-SSR_P7.62mm_Straight, symbol Relay_SolidState:S102S01
- removed U6: LM7805_TO220, Package_TO_SOT_THT:TO-220F-3_Horizontal_TabDown, symbol Regulator_Linear:LM7805_TO220
- added D1: 1N5819WS, Diode_SMD:D_SOD-323, symbol Diode:1N5819WS
- added K1: G5NB-1A-E DC12, G5NB-1A-E_DC12:RELAY_G5NB-1A_DC5_OMR, symbol G5NB-1A-E_DC12:G5NB-1A-E_DC12
- added U1: TPS63070RNMR, TPS63070RNMR:VREG_TPS63070RNMR, symbol TPS63070RNMR:TPS63070RNMR
- added U3: AMS1117-5.0, Package_TO_SOT_SMD:SOT-223-3_TabPin2, symbol Regulator_Linear:AMS1117-5.0
- added U6: MAX17048G_T10, MAX17048G_T10:SON50P200X200X80-9N, symbol MAX17048G_T10:MAX17048G_T10
- U9: footprint Package_SIP:SIP4_Sharp-SSR_P7.62mm_Straight -> G5NB-1A-E_DC12:RELAY_G5NB-1A_DC5_OMR; symbol Relay_SolidState:S102S01 -> G5NB-1A-E_DC12:G5NB-1A-E_DC12; Availability (none) -> In Stock; COPYRIGHT (none) -> Copyright (C) 2023 Ultra Librarian. All rights reserved.; Check_prices (none) -> https://www.snapeda.com/parts/G5NB-1A-E%20DC12/Omron+Electr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; MANUFACTURER_PART_NUMBER (none) -> G5NB-1A-E DC12; MF (none) -> Omron Electronics Inc-EMC Div; MFR_NAME (none) -> Omron; MP (none) -> G5NB-1A-E DC12; Package (none) -> None; Price (none) -> None; Purchase-URL (none) -> https://www.snapeda.com/api/url_track_click_mouser/?unipart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; SnapEDA_Link (none) -> https://www.snapeda.com/parts/G5NB-1A-E%20DC12/Omron+Electr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
- renumbered C7 to C3, C4 to C5, C5 to C6, C6 to C7, D3 to D9, J2 to J1, U1 to U2, U4 to U7
Connections:
- net +12V: now also U9.4, D1.2 (A), K1.4, U3.3 (VI); no longer U9.3
- net +3.3V: now also R18.2; no longer R18.1
- net +5V: now also U3.2 (VO)
- net Buck_In: now also D1.1 (K)
- net GND: now also U3.1 (GND), U6.1 (CTG), U6.4 (GND), U6.9 (EP)
- net MCU_BAT: now also U6.2 (CELL)
- net SCL: now also U6.7 (SCL)
- net SDA: now also R18.1, U6.8 (SDA); no longer R18.2
- net at J4.1 (Pin_1), J4.2 (Pin_2): now also K1.2
- net at J6.1 (Pin_1), J6.2 (Pin_2): now also K1.3
- net at Q2.1 (D): now also K1.1
- net at L1.1: now also U1.9 (L2); no longer U4.11 (L1)
- net at L1.2: now also U1.11 (L1); no longer U4.9 (L2)
- net at R22.2: now also U6.5 (~{ALERT})
- net at Q3.1 (D): now also U9.1; no longer U9.4
- net at R17.1: now also U6.6 (QSTRT)
- net at JP1.2 (C): now also U6.3 (VDD)
- net at J3.2 (Pin_2): now also U9.3; no longer U9.1
Other:
- moved on the sheet: J3, L1, Q3, R17, R18, R19, R22, R6, R9, SW1

Commit message: improved schematic
Parts:
- removed U4: ~, Package_DFN_QFN:TDFN-8-1EP_2x2mm_P0.5mm_EP0.8x1.2mm, symbol Custom:TPS63070
- added C10: 10u, Capacitor_SMD:C_0402_1005Metric, symbol Device:C
Connections:
- net +3.3V: now also U1.7_8 (VOUT), C10.2
- net EN: now also U1.14 (EN)
- net GND: now also U1.10 (PGND), U1.15 (VSEL), U1.2 (PG), U1.4 (GND), U1.6 (FB2), C10.1
- net PS: now also U1.1 (PS/SYNC)
- net TPS_VIN: now reaches U1.12_13 (VIN)
- net TPS_VIN: now also C1.1, C13.1, C2.1, C8.1, JP2.2 (B), R23.1, R24.1
- net TPS_VAUX: now reaches U1.3 (VAUX)
- net TPS_VAUX: now also C14.1
- net TPS_FB: now reaches U1.5 (FB)
- net TPS_FB: now also R25.1, R30.2
Other:
- moved on the sheet: L1

Commit message: first revision of pcb ready. very crude.. needs another looky
Parts:
- removed JP1: Jumper_3_Bridged12, Jumper:SolderJumper-3_P1.3mm_Bridged2Bar12_Pad1.0x1.5mm_NumberLabels, symbol Jumper:Jumper_3_Bridged12
- removed SW4: SW, Button_Switch_SMD:Nidec_Copal_CAS-120A, symbol Switch:SW_Nidec_CAS-120A1
- J16: value Rotary_Encoder -> Conn_01x05; footprint Connector_JST:JST_GH_SM03B-GHS-TB_1x03-1MP_P1.25mm_Horizontal -> Connector_JST:JST_GH_BM05B-GHS-TBT_1x05-1MP_P1.25mm_Vertical
- J8: footprint Connector_JST:JST_GH_SM02B-GHS-TB_1x02-1MP_P1.25mm_Horizontal -> Connector_JST:JST_EH_S2B-EH_1x02_P2.50mm_Horizontal
- SW1: value SW_MEC_5G -> SW_Omron_B3FS; footprint Button_Switch_SMD:SW_SPST_B3U-1000P -> Button_Switch_SMD:SW_SPST_B3U-1000P-B; symbol Switch:SW_MEC_5G -> Switch:SW_Omron_B3FS
- SW2: value SW_MEC_5G -> SW_Omron_B3FS; symbol Switch:SW_MEC_5G -> Switch:SW_Omron_B3FS
Connections:
- net GND: no longer SW1.2 (A), SW2.2 (A)
- net GPIO0: now also SW1.2; no longer SW1.3 (B), SW1.4 (B)
- net MCU_BAT: now also J14.2, U6.3 (VDD)
- net P_IO_4: no longer J20.3 (Pin_3), U5.10 (P5)
- net RESET: now also SW2.2; no longer SW2.3 (B), SW2.4 (B)
- new net P_IO_7: J20.3 (Pin_3), U5.10 (P5)
- no-connect marks 8 -> 7
Other:
- note removed: "tps63070"
- moved on the sheet: C3, J16, R1, SW1, SW2
